File: DigitDisplay1.sch (KiCad schematic (older format))
At the start: 18 parts, among them U2 74HC164

Commit message: add the RTC module and base prototype pcb layout
Parts:
- C2: footprint (none) -> Capacitor_THT:C_Disc_D3.4mm_W2.1mm_P2.50mm
- R11, R12, R13: footprint Resistor_SMD:R_0201_0603Metric -> Resistor_SMD:R_0805_2012Metric
Changed lines of the file:
@@
 F 0 "R13" V 8050 3000 50  0000 C CNN
 F 1 "150R" V 7900 2850 50  0000 C CNN
-F 2 "Resistor_SMD:R_0201_0603Metric" V 7930 2850 50  0001 C CNN
+F 2 "Resistor_SMD:R_0805_2012Metric" V 7930 2850 50  0001 C CNN
 F 3 "~" H 8000 2850 50  0001 C CNN
 	1    8000 2850
@@
 F 0 "R12" V 7500 3000 50  0000 C CNN
 F 1 "150R" V 7350 2850 50  0000 C CNN
-F 2 "Resistor_SMD:R_0201_0603Metric" V 7380 2850 50  0001 C CNN
+F 2 "Resistor_SMD:R_0805_2012Metric" V 7380 2850 50  0001 C CNN
 F 3 "~" H 7450 2850 50  0001 C CNN
 	1    7450 2850
@@
 F 0 "R11" V 6950 3000 50  0000 C CNN
 F 1 "150R" V 6800 2850 50  0000 C CNN
-F 2 "Resistor_SMD:R_0201_0603Metric" V 6830 2850 50  0001 C CNN
+F 2 "Resistor_SMD:R_0805_2012Metric" V 6830 2850 50  0001 C CNN
 F 3 "~" H 6900 2850 50  0001 C CNN
 	1    6900 2850
@@
 F 0 "C2" H 1800 4200 50  0000 L CNN
 F 1 "100nF" H 1800 4150 50  0000 L CNN
-F 2 "" H 1688 4000 50  0001 C CNN
+F 2 "Capacitor_THT:C_Disc_D3.4mm_W2.1mm_P2.50mm" H 1688 4000 50  0001 C CNN
 F 3 "~" H 1650 4150 50  0001 C CNN
 	1    1650 4150
