File: DigitDisplay2.sch (KiCad schematic (older format))
At the start: 18 parts, among them U3 74HC164

Commit message: add the RTC module and base prototype pcb layout
Parts:
- C3: footprint (none) -> Capacitor_THT:C_Disc_D3.4mm_W2.1mm_P2.50mm
- R14, R15, R16: footprint Resistor_SMD:R_0201_0603Metric -> Resistor_SMD:R_0805_2012Metric
Changed lines of the file:
@@
 F 0 "R16" V 8050 3000 50  0000 C CNN
 F 1 "150R" V 7900 2850 50  0000 C CNN
-F 2 "Resistor_SMD:R_0201_0603Metric" V 7930 2850 50  0001 C CNN
+F 2 "Resistor_SMD:R_0805_2012Metric" V 7930 2850 50  0001 C CNN
 F 3 "~" H 8000 2850 50  0001 C CNN
 	1    8000 2850
@@
 F 0 "R15" V 7500 3000 50  0000 C CNN
 F 1 "150R" V 7350 2850 50  0000 C CNN
-F 2 "Resistor_SMD:R_0201_0603Metric" V 7380 2850 50  0001 C CNN
+F 2 "Resistor_SMD:R_0805_2012Metric" V 7380 2850 50  0001 C CNN
 F 3 "~" H 7450 2850 50  0001 C CNN
 	1    7450 2850
@@
 F 0 "R14" V 6950 3000 50  0000 C CNN
 F 1 "150R" V 6800 2850 50  0000 C CNN
-F 2 "Resistor_SMD:R_0201_0603Metric" V 6830 2850 50  0001 C CNN
+F 2 "Resistor_SMD:R_0805_2012Metric" V 6830 2850 50  0001 C CNN
 F 3 "~" H 6900 2850 50  0001 C CNN
 	1    6900 2850
@@
 F 0 "C3" H 2300 4200 50  0000 L CNN
 F 1 "100nF" H 2300 4150 50  0000 L CNN
-F 2 "" H 2188 4000 50  0001 C CNN
+F 2 "Capacitor_THT:C_Disc_D3.4mm_W2.1mm_P2.50mm" H 2188 4000 50  0001 C CNN
 F 3 "~" H 2150 4150 50  0001 C CNN
 	1    2150 4150
